Commit message: slam functionality working, gps drifting still

File: ark_rover/description/robot_core.xacro (robot description, xacro)
@@ -17,4 +17,12 @@
 <!-- BASE LINK -->
 <link name="base_link">
+</link>
+<!-- BASE_FOOTPRINT LINK -->
+<joint name="base_footprint_joint" type="fixed">
+    <parent link="base_link"/>
+    <child link="base_footprint"/>
+    <origin xyz="0 0 0" rpy="0 0 0"/>
+</joint>
+<link name="base_footprint">
 </link>
 <!--

Commit message: urdf changes, foxglove instead of rviz, battery publisher

File: ark_rover/description/robot_core.xacro (robot description, xacro)
@@ -25,4 +25,12 @@
 </joint>
 <link name="base_footprint">
+</link>
+<!-- CAMERA LINK -->
+<joint name="oak-d-base-frame_joint" type="fixed">
+    <parent link="base_link"/>
+    <child link="oak-d-base-frame"/>
+    <origin xyz="0.158 0 0.120" rpy="0 0 0"/>
+</joint>
+<link name="oak-d-base-frame">
 </link>
 <!--
